File: Hardware/SparkFun_Qwiic_CO2_Sensor_XENSIV_PAS.brd (EAGLE design)
At the start: 25.4 x 40.6 mm, 71 parts, among them J1 QWIIC_RA, J2 QWIIC_RA, U1 PASCO2V01BUMA1, U2 LMR62421

Commit message: Update pre design review
Add keepouts for exposed pads.
Move vias to avoid keepouts.
Add 10k PUR to PSEL 3.3V selector.
Add voltage/current details to CO2 sensor on schematic.
Modified bottom PTHs to match standard order.
Move vias for ground pour.
Remove ground stub and unnecessary tRestrict.
Parts:
- added R7: 10k, SparkFun-Resistors:0603
- U$16: device output:#_SDA#TX#0 -> output:#_SDA#0
- U$20: device output:#_3V3#0 -> output:#_SDA#TX#0
- moved U$14 7.62 mm to (15.2, 1.27)
- moved U$18 7.62 mm to (15.2, 1.27)
- moved U$20 5.08 mm to (10.2, 1.27)
- moved U$19 2.54 mm to (12.7, 1.27)
- moved U$15 2.54 mm to (7.62, 1.27)
- moved U$17 2.54 mm to (7.62, 1.27)
- moved R6 2.54 mm to (12.7, 39.2)
- moved U$16 2.54 mm to (10.2, 1.27)
- moved U$29 1.52 mm to (20.3, 39.2)
- moved D2 1.52 mm to (16.8, 39.2)
- moved C8 0.13 mm to (2.54, 37.0)
- moved C7 0.13 mm to (4.57, 37.0)
Connections:
- new net N$8: PSEL.1, R7.1
- net 3.3V: now also J4.3, R7.2; no longer J4.2, PSEL.1
- net GND: now also J4.2; no longer J4.5
- net SCL: now also J4.5; no longer J4.4
- net SDA/TX: now also J4.4; no longer J4.3
Routing:
- net N$8: track 0.00 -> 8.42 mm, vias 0 -> 1
- net 3.3V: track 85.9 -> 91.2 mm
- net N$7: track 5.29 -> 2.75 mm
- net GND: track 0.00 -> 1.91 mm, vias 71 -> 66
- net SDA/TX: track 59.6 -> 61.1 mm
- net N$6: track 3.35 -> 2.34 mm
