File: Hardware/SparkFun_Qwiic_CO2_Sensor_XENSIV_PAS.brd (EAGLE design)
At the start: 25.4 x 40.6 mm, 79 parts, among them J1 QWIIC_RA, J2 QWIIC_RA, U1 PASCO2V01BUMA1, U2 LMR62421

Commit message: BOM change and add logo to silk.
Parts:
- added U$23: (no value), xensiv_pas:INFINEON_LOGO
- R3: value 1M -> 100k
- U2: value LMR62421 -> AP3012
Changed lines of the file:
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@@
 <drawing>
 <settings>
-<setting alwaysvectorfont="yes"/>
+<setting alwaysvectorfont="no"/>
 <setting verticaltext="up"/>
 </settings>
-<grid distance="0.005" unitdist="inch" unit="inch" style="lines" multiple="1" display="yes" altdistance="0.001" altunitdist="inch" altunit="inch"/>
+<grid distance="0.01" unitdist="mm" unit="mm" style="lines" multiple="1" display="yes" altdistance="0.005" altunitdist="mm" altunit="mm"/>
 <layers>
 <layer number="1" name="Top" color="4" fill="1" visible="yes" active="yes"/>
@@
 <layer number="28" name="bValues" color="7" fill="1" visible="no" active="yes"/>
 <layer number="29" name="tStop" color="7" fill="3" visible="no" active="yes"/>
-<layer number="30" name="bStop" color="7" fill="6" visible="no" active="yes"/>
+<layer number="30" name="bStop" color="7" fill="6" visible="yes" active="yes"/>
 <layer number="31" name="tCream" color="7" fill="4" visible="no" active="yes"/>
 <layer number="32" name="bCream" color="7" fill="5" visible="no" active="yes"/>
@@
 <attribute name="VALUE" x="23.622" y="11.049" size="0.6096" layer="27" font="vector" ratio="20" rot="R90"/>
 </element>
-<element name="U2" library="xensiv_pas" package="SOT95P280X145-5M" package3d_urn="urn:adsk.eagle:package:40937508/1" value="LMR62421" x="12.7" y="11.43" smashed="yes">
+<element name="U2" library="xensiv_pas" package="SOT95P280X145-5M" package3d_urn="urn:adsk.eagle:package:40937508/1" value="AP3012" x="12.7" y="11.43" smashed="yes">
 <attribute name="NAME" x="12.7" y="14.0836" size="1.27" layer="25" align="bottom-center"/>
-<attribute name="PROD_ID" value="VREG-19362" x="12.7" y="11.43" size="1.778" layer="27" display="off"/>
-<attribute name="VALUE" x="12.7" y="9.2164" size="1.27" layer="27" align="top-center"/>
+<attribute name="PN" value="AP3012" x="12.7" y="11.43" size="1.778" layer="27" display="off"/>
+<attribute name="PROD_ID" value="VREG-13911" x="12.7" y="11.43" size="1.778" layer="27" display="off"/>
+<attribute name="VALUE" value="AP3012" x="12.7" y="11.43" size="1.778" layer="27" display="off"/>
 </element>
 <element name="C1" library="SparkFun-Capacitors" package="0805" value="10uF" x="17.526" y="13.208" smashed="yes" rot="R90">
@@
 <attribute name="VALUE" x="9.779" y="13.843" size="0.6096" layer="27" font="vector" ratio="20" align="top-center"/>
 </element>
-<element name="R3" library="SparkFun-Resistors" package="0603" value="1M" x="15.875" y="11.43" smashed="yes" rot="R90">
+<element name="R3" library="SparkFun-Resistors" package="0603" value="100k" x="15.875" y="11.43" smashed="yes" rot="R90">
 <attribute name="NAME" x="15.113" y="11.43" size="0.6096" layer="25" font="vector" ratio="20" rot="R90" align="bottom-center"/>
-<attribute name="PROD_ID" value="RES-07868" x="15.875" y="11.43" size="1.778" layer="27" rot="R90" display="off"/>
-<attribute name="VALUE" x="16.637" y="11.43" size="0.6096" layer="27" font="vector" ratio="20" rot="R90" align="top-center"/>
+<attribute name="PROD_ID" value="RES-07828" x="15.875" y="11.43" size="1.778" layer="27" rot="R90" display="off"/>
+<attribute name="VALUE" value="100k" x="16.637" y="11.43" size="0.6096" layer="27" font="vector" ratio="20" rot="R90" align="top-center"/>
 </element>
 <element name="LOGO1" library="SparkFun-Aesthetics" package="SFE_LOGO_NAME_FLAME_.1" value="SFE_LOGO_NAME_FLAME.1_INCH" x="12.7" y="17.272" smashed="yes" rot="MR0"/>
@@
 <element name="U$25" library="output" package="CO2_SENSOR0" value="" x="12.7" y="11.938" smashed="yes" rot="MR0"/>
 <element name="U$39" library="output" package="PASCO2V010" value="" x="12.7" y="10.287" smashed="yes" rot="MR0"/>
+<element name="U$23" library="xensiv_pas" package="INFINEON_LOGO" value="" x="7.58" y="37.36" smashed="yes" rot="MR0"/>
 </elements>
 <signals>
