File: Production/SparkFun_Qwiic_CO2_Sensor_XENSIV_PAS-Panel.brd (EAGLE design)
At the start: 175 x 96 mm, 930 parts, among them J1 QWIIC_RA, J11 QWIIC_RA, J12 QWIIC_RA, J16 QWIIC_RA, J17 QWIIC_RA, J2 QWIIC_RA, J21 QWIIC_RA, J22 QWIIC_RA, J26 QWIIC_RA, J27 QWIIC_RA, J31 QWIIC_RA, J32 QWIIC_RA, J36 QWIIC_RA, J37 QWIIC_RA, J41 QWIIC_RA, J42 QWIIC_RA, J46 QWIIC_RA, J47 QWIIC_RA, J51 QWIIC_RA, J52 QWIIC_RA, J56 QWIIC_RA, J57 QWIIC_RA, J6 QWIIC_RA, J7 QWIIC_RA, U1 PASCO2V01BUMA1, U10 LMR62421, U11 PASCO2V01BUMA1, U12 LMR62421, U13 PASCO2V01BUMA1, U14 LMR62421, U15 PASCO2V01BUMA1, U16 LMR62421, U17 PASCO2V01BUMA1, U18 LMR62421, U19 PASCO2V01BUMA1, U2 LMR62421, U20 LMR62421, U21 PASCO2V01BUMA1, U22 LMR62421, U23 PASCO2V01BUMA1, U24 LMR62421, U3 PASCO2V01BUMA1, U4 LMR62421, U5 PASCO2V01BUMA1, U6 LMR62421, U7 PASCO2V01BUMA1, U8 LMR62421, U9 PASCO2V01BUMA1

Commit message: Move Flame silk to middle.
Repanelize after.
Parts:
- moved U$149 14.7 mm to (116.3, 7.62)
- moved U$371 14.7 mm to (116.3, 48.8)
- moved U$1 14.7 mm to (12.7, 7.62)
- moved U$223 14.7 mm to (12.7, 48.8)
- moved U$23 14.7 mm to (38.6, 7.62)
- moved U$260 14.7 mm to (38.6, 48.8)
- moved U$112 14.7 mm to (90.4, 7.62)
- moved U$186 14.7 mm to (142.2, 7.62)
- moved U$297 14.7 mm to (64.5, 48.8)
- moved U$334 14.7 mm to (90.4, 48.8)
- moved U$408 14.7 mm to (142.2, 48.8)
- moved U$75 14.7 mm to (64.5, 7.62)
Changed lines of the file:
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@@
 <attribute name="VALUE" x="22.098" y="33.02" size="0.6096" layer="27" font="vector" ratio="20" rot="R270"/>
 </element>
-<element name="U$1" library="SparkFun-Aesthetics" package="SFE_LOGO_FLAME_.1" value="" x="22.86" y="18.288" smashed="yes"/>
+<element name="U$1" library="SparkFun-Aesthetics" package="SFE_LOGO_FLAME_.1" value="" x="12.7" y="7.62" smashed="yes"/>
 <element name="U$4" library="output" package="#GND_#0" value="" x="24.13" y="29.21" smashed="yes"/>
 <element name="U$5" library="output" package="#GND_#0" value="" x="1.27" y="29.21" smashed="yes" rot="MR0"/>
@@
 <attribute name="VALUE" x="48.006" y="33.02" size="0.6096" layer="27" font="vector" ratio="20" rot="R270"/>
 </element>
-<element name="U$23" library="SparkFun-Aesthetics" package="SFE_LOGO_FLAME_.1" value="" x="48.768" y="18.288" smashed="yes"/>
+<element name="U$23" library="SparkFun-Aesthetics" package="SFE_LOGO_FLAME_.1" value="" x="38.608" y="7.62" smashed="yes"/>
 <element name="U$30" library="output" package="#GND_#0" value="" x="50.038" y="29.21" smashed="yes"/>
 <element name="U$40" library="output" package="#GND_#0" value="" x="27.178" y="29.21" smashed="yes" rot="MR0"/>
@@
 <attribute name="VALUE" x="73.914" y="33.02" size="0.6096" layer="27" font="vector" ratio="20" rot="R270"/>
 </element>
-<element name="U$75" library="SparkFun-Aesthetics" package="SFE_LOGO_FLAME_.1" value="" x="74.676" y="18.288" smashed="yes"/>
+<element name="U$75" library="SparkFun-Aesthetics" package="SFE_LOGO_FLAME_.1" value="" x="64.516" y="7.62" smashed="yes"/>
 <element name="U$76" library="output" package="#GND_#0" value="" x="75.946" y="29.21" smashed="yes"/>
 <element name="U$77" library="output" package="#GND_#0" value="" x="53.086" y="29.21" smashed="yes" rot="MR0"/>
@@
 <attribute name="VALUE" x="99.822" y="33.02" size="0.6096" layer="27" font="vector" ratio="20" rot="R270"/>
 </element>
-<element name="U$112" library="SparkFun-Aesthetics" package="SFE_LOGO_FLAME_.1" value="" x="100.584" y="18.288" smashed="yes"/>
+<element name="U$112" library="SparkFun-Aesthetics" package="SFE_LOGO_FLAME_.1" value="" x="90.424" y="7.62" smashed="yes"/>
 <element name="U$113" library="output" package="#GND_#0" value="" x="101.854" y="29.21" smashed="yes"/>
 <element name="U$114" library="output" package="#GND_#0" value="" x="78.994" y="29.21" smashed="yes" rot="MR0"/>
@@
 <attribute name="VALUE" x="125.73" y="33.02" size="0.6096" layer="27" font="vector" ratio="20" rot="R270"/>
 </element>
-<element name="U$149" library="SparkFun-Aesthetics" package="SFE_LOGO_FLAME_.1" value="" x="126.492" y="18.288" smashed="yes"/>
+<element name="U$149" library="SparkFun-Aesthetics" package="SFE_LOGO_FLAME_.1" value="" x="116.332" y="7.62" smashed="yes"/>
 <element name="U$150" library="output" package="#GND_#0" value="" x="127.762" y="29.21" smashed="yes"/>
 <element name="U$151" library="output" package="#GND_#0" value="" x="104.902" y="29.21" smashed="yes" rot="MR0"/>
@@
 <attribute name="VALUE" x="151.638" y="33.02" size="0.6096" layer="27" font="vector" ratio="20" rot="R270"/>
 </element>
-<element name="U$186" library="SparkFun-Aesthetics" package="SFE_LOGO_FLAME_.1" value="" x="152.4" y="18.288" smashed="yes"/>
+<element name="U$186" library="SparkFun-Aesthetics" package="SFE_LOGO_FLAME_.1" value="" x="142.24" y="7.62" smashed="yes"/>
 <element name="U$187" library="output" package="#GND_#0" value="" x="153.67" y="29.21" smashed="yes"/>
 <element name="U$188" library="output" package="#GND_#0" value="" x="130.81" y="29.21" smashed="yes" rot="MR0"/>
@@
 <attribute name="VALUE" x="22.098" y="74.168" size="0.6096" layer="27" font="vector" ratio="20" rot="R270"/>
 </element>
-<element name="U$223" library="SparkFun-Aesthetics" package="SFE_LOGO_FLAME_.1" value="" x="22.86" y="59.436" smashed="yes"/>
+<element name="U$223" library="SparkFun-Aesthetics" package="SFE_LOGO_FLAME_.1" value="" x="12.7" y="48.768" smashed="yes"/>
 <element name="U$224" library="output" package="#GND_#0" value="" x="24.13" y="70.358" smashed="yes"/>
 <element name="U$225" library="output" package="#GND_#0" value="" x="1.27" y="70.358" smashed="yes" rot="MR0"/>
@@
 <attribute name="VALUE" x="48.006" y="74.168" size="0.6096" layer="27" font="vector" ratio="20" rot="R270"/>
 </element>
-<element name="U$260" library="SparkFun-Aesthetics" package="SFE_LOGO_FLAME_.1" value="" x="48.768" y="59.436" smashed="yes"/>
+<element name="U$260" library="SparkFun-Aesthetics" package="SFE_LOGO_FLAME_.1" value="" x="38.608" y="48.768" smashed="yes"/>
 <element name="U$261" library="output" package="#GND_#0" value="" x="50.038" y="70.358" smashed="yes"/>
 <element name="U$262" library="output" package="#GND_#0" value="" x="27.178" y="70.358" smashed="yes" rot="MR0"/>
@@
 <attribute name="VALUE" x="73.914" y="74.168" size="0.6096" layer="27" font="vector" ratio="20" rot="R270"/>
 </element>
-<element name="U$297" library="SparkFun-Aesthetics" package="SFE_LOGO_FLAME_.1" value="" x="74.676" y="59.436" smashed="yes"/>
+<element name="U$297" library="SparkFun-Aesthetics" package="SFE_LOGO_FLAME_.1" value="" x="64.516" y="48.768" smashed="yes"/>
 <element name="U$298" library="output" package="#GND_#0" value="" x="75.946" y="70.358" smashed="yes"/>
 <element name="U$299" library="output" package="#GND_#0" value="" x="53.086" y="70.358" smashed="yes" rot="MR0"/>
@@
 <attribute name="VALUE" x="99.822" y="74.168" size="0.6096" layer="27" font="vector" ratio="20" rot="R270"/>
 </element>
-<element name="U$334" library="SparkFun-Aesthetics" package="SFE_LOGO_FLAME_.1" value="" x="100.584" y="59.436" smashed="yes"/>
+<element name="U$334" library="SparkFun-Aesthetics" package="SFE_LOGO_FLAME_.1" value="" x="90.424" y="48.768" smashed="yes"/>
 <element name="U$335" library="output" package="#GND_#0" value="" x="101.854" y="70.358" smashed="yes"/>
 <element name="U$336" library="output" package="#GND_#0" value="" x="78.994" y="70.358" smashed="yes" rot="MR0"/>
@@
 <attribute name="VALUE" x="125.73" y="74.168" size="0.6096" layer="27" font="vector" ratio="20" rot="R270"/>
 </element>
-<element name="U$371" library="SparkFun-Aesthetics" package="SFE_LOGO_FLAME_.1" value="" x="126.492" y="59.436" smashed="yes"/>
+<element name="U$371" library="SparkFun-Aesthetics" package="SFE_LOGO_FLAME_.1" value="" x="116.332" y="48.768" smashed="yes"/>
 <element name="U$372" library="output" package="#GND_#0" value="" x="127.762" y="70.358" smashed="yes"/>
 <element name="U$373" library="output" package="#GND_#0" value="" x="104.902" y="70.358" smashed="yes" rot="MR0"/>
@@
 <attribute name="VALUE" x="151.638" y="74.168" size="0.6096" layer="27" font="vector" ratio="20" rot="R270"/>
 </element>
-<element name="U$408" library="SparkFun-Aesthetics" package="SFE_LOGO_FLAME_.1" value="" x="152.4" y="59.436" smashed="yes"/>
+<element name="U$408" library="SparkFun-Aesthetics" package="SFE_LOGO_FLAME_.1" value="" x="142.24" y="48.768" smashed="yes"/>
 <element name="U$409" library="output" package="#GND_#0" value="" x="153.67" y="70.358" smashed="yes"/>
 <element name="U$410" library="output" package="#GND_#0" value="" x="130.81" y="70.358" smashed="yes" rot="MR0"/>

Commit message: BOM change and add logo to silk.
Parts:
- added U$445: (no value), output:#P_#0
- added U$446: (no value), output:#_PWM#0
- added U$447: (no value), output:#PWM#0
- added U$448: (no value), output:#PWR#0
- added U$449, U$450: (no value), output:#_SDA#0
- added U$451: (no value), output:#_SCL#0
- added U$452: (no value), output:PHOTOACOUSTIC0
- added U$453: (no value), output:SPECTROSCOPY0
- added U$454: (no value), output:CO2_SENSOR0
- added U$455: (no value), output:PASCO2V010
- added U$456: (no value), xensiv_pas:INFINEON_LOGO
- R10, R17, R24, R3, R31, R38, R45, R52, R59, R66, R73, R80: value 1M -> 100k
- U$100, U$63: device output:#_3V3#0 -> output:#_EN#0
- U$101, U$138: device output:#P_#0 -> output:#_EN#0
- U$102: device output:#_PWM#0 -> output:#_3V3#0
- U$103: device output:#PWM#0 -> output:#P_#0
- U$104: device output:#PWR#0 -> output:#_PWM#0
- U$105, U$143: device output:#_SDA#0 -> output:#PWM#0
- U$106, U$68: device output:#_SDA#0 -> output:#PWR#0
- U$107, U$70: device output:#_SCL#0 -> output:#_SDA#0
- U$108, U$145: device output:PHOTOACOUSTIC0 -> output:#_SDA#0
- U$109: device output:SPECTROSCOPY0 -> output:#_SCL#0
- U$110: device output:CO2_SENSOR0 -> output:PHOTOACOUSTIC0
- U$111: device output:PASCO2V010 -> output:SPECTROSCOPY0
- U$112: device SparkFun-Aesthetics:SFE_LOGO_FLAME_.1 -> output:CO2_SENSOR0
- U$113, U$151: device output:#GND_#0 -> output:PASCO2V010
- U$114, U$76: device output:#GND_#0 -> xensiv_pas:INFINEON_LOGO
- U$115: device output:#_TX#0 -> SparkFun-Aesthetics:SFE_LOGO_FLAME_.1
- U$116, U$79: device output:#_RX#0 -> output:#GND_#0
- U$117, U$154, U$155, U$192, U$269, U$306, U$345, U$382: device output:#_GND#0 -> output:#GND_#0
- U$118, U$232, U$308, U$80: device output:#_GND#0 -> output:#_TX#0
- U$119: device output:#RX_#0 -> output:#_RX#0
- U$120, U$83: device output:#SDA#TX_#0 -> output:#_GND#0
- U$122: device output:#_SCL#0 -> output:#RX_#0
- U$123, U$47: device output:#_GND#0 -> output:#SDA#TX_#0
- U$124, U$235, U$272, U$50: device output:#_3V3#0 -> output:#_GND#0
- U$125, U$163: device output:#_INT#0 -> output:#_SCL#0
- U$126, U$162, U$200, U$273, U$310, U$311, U$348, U$88: device output:#_INT#0 -> output:#_GND#0
- U$127: device output:#PSEL#0 -> output:#_3V3#0
- U$128, U$91: device output:#I�C#0 -> output:#_INT#0
- U$129, U$166: device SparkFun-Aesthetics:SFE_LOGO_FLAME_STOP_.1 -> output:#_INT#0
- U$130: device output:PWR0 -> output:#PSEL#0
- U$131: device output:#U#0 -> output:#I�C#0
- U$132: device output:#I#0 -> SparkFun-Aesthetics:SFE_LOGO_FLAME_STOP_.1
- U$133: device output:#12VI_#0 -> output:PWR0
- U$134: device output:#_12VIN#0 -> output:#U#0
- U$135, U$173: device output:#_EN#0 -> output:#I#0
- U$136, U$98: device output:#_EN#0 -> output:#12VI_#0
- U$137: device output:#_3V3#0 -> output:#_12VIN#0
- U$139, U$176: device output:#_PWM#0 -> output:#_EN#0
- U$140: device output:#PWM#0 -> output:#_3V3#0
- U$141: device output:#PWR#0 -> output:#P_#0
- U$142, U$180: device output:#_SDA#0 -> output:#_PWM#0
- U$144: device output:#_SCL#0 -> output:#PWR#0
- U$146, U$183: device output:SPECTROSCOPY0 -> output:#_SDA#0
- U$147: device output:CO2_SENSOR0 -> output:#_SCL#0
- U$148: device output:PASCO2V010 -> output:PHOTOACOUSTIC0
- U$149: device SparkFun-Aesthetics:SFE_LOGO_FLAME_.1 -> output:SPECTROSCOPY0
- U$150, U$188: device output:#GND_#0 -> output:CO2_SENSOR0
- U$152: device output:#_TX#0 -> xensiv_pas:INFINEON_LOGO
- U$153: device output:#_RX#0 -> SparkFun-Aesthetics:SFE_LOGO_FLAME_.1
- U$156: device output:#RX_#0 -> output:#_TX#0
- U$157: device output:#SDA#TX_#0 -> output:#_RX#0
- U$159, U$196, U$48: device output:#_SCL#0 -> output:#_GND#0
- U$160, U$84: device output:#_GND#0 -> output:#RX_#0
- U$161: device output:#_3V3#0 -> output:#SDA#TX_#0
- U$164, U$238, U$349, U$386: device output:#PSEL#0 -> output:#_GND#0
- U$165: device output:#I�C#0 -> output:#_3V3#0
- U$167, U$204: device output:PWR0 -> output:#_INT#0
- U$168: device output:#U#0 -> output:#PSEL#0
- U$169: device output:#I#0 -> output:#I�C#0
- U$170: device output:#12VI_#0 -> SparkFun-Aesthetics:SFE_LOGO_FLAME_STOP_.1
- U$171: device output:#_12VIN#0 -> output:PWR0
- U$172, U$210: device output:#_EN#0 -> output:#U#0
- U$174: device output:#_3V3#0 -> output:#12VI_#0
- U$175: device output:#P_#0 -> output:#_12VIN#0
- U$177, U$214: device output:#PWM#0 -> output:#_EN#0
- U$178: device output:#PWR#0 -> output:#_3V3#0
- U$179, U$217: device output:#_SDA#0 -> output:#P_#0
- U$181: device output:#_SCL#0 -> output:#PWM#0
- U$182: device output:PHOTOACOUSTIC0 -> output:#PWR#0
- U$184, U$221: device output:CO2_SENSOR0 -> output:#_SDA#0
- U$185: device output:PASCO2V010 -> output:#_SCL#0
- U$186: device SparkFun-Aesthetics:SFE_LOGO_FLAME_.1 -> output:PHOTOACOUSTIC0
- U$187, U$225: device output:#GND_#0 -> output:SPECTROSCOPY0
- U$189: device output:#_TX#0 -> output:PASCO2V010
- U$190: device output:#_RX#0 -> xensiv_pas:INFINEON_LOGO
- U$191, U$229, U$343, U$419: device output:#_GND#0 -> SparkFun-Aesthetics:SFE_LOGO_FLAME_.1
- U$193, U$230: device output:#RX_#0 -> output:#GND_#0
- U$194: device output:#SDA#TX_#0 -> output:#_TX#0
- U$195, U$271, U$43, U$81: device output:#_GND#0 -> output:#_RX#0
- U$198: device output:#_3V3#0 -> output:#RX_#0
- U$199, U$237: device output:#_INT#0 -> output:#SDA#TX_#0
- U$201: device output:#PSEL#0 -> output:#_SCL#0
- U$202, U$276, U$387, U$424: device output:#I�C#0 -> output:#_GND#0
- U$203: device SparkFun-Aesthetics:SFE_LOGO_FLAME_STOP_.1 -> output:#_3V3#0
- U$205, U$242: device output:#U#0 -> output:#_INT#0
- U$206: device output:#I#0 -> output:#PSEL#0
- U$207: device output:#12VI_#0 -> output:#I�C#0
- U$208: device output:#_12VIN#0 -> SparkFun-Aesthetics:SFE_LOGO_FLAME_STOP_.1
- U$209, U$247: device output:#_EN#0 -> output:PWR0
- U$211: device output:#_3V3#0 -> output:#I#0
- U$212: device output:#P_#0 -> output:#12VI_#0
- U$213: device output:#_PWM#0 -> output:#_12VIN#0
- U$215, U$252: device output:#PWR#0 -> output:#_EN#0
- U$216, U$254: device output:#_SDA#0 -> output:#_3V3#0
- U$218: device output:#_SCL#0 -> output:#_PWM#0
- U$219: device output:PHOTOACOUSTIC0 -> output:#PWM#0
- U$220: device output:SPECTROSCOPY0 -> output:#PWR#0
- U$222, U$259: device output:PASCO2V010 -> output:#_SDA#0
- U$223: device SparkFun-Aesthetics:SFE_LOGO_FLAME_.1 -> output:#_SCL#0
- U$224, U$262: device output:#GND_#0 -> output:PHOTOACOUSTIC0
- U$226: device output:#_TX#0 -> output:CO2_SENSOR0
- U$227: device output:#_RX#0 -> output:PASCO2V010
- U$228, U$266, U$380: device output:#_GND#0 -> xensiv_pas:INFINEON_LOGO
- U$23: device SparkFun-Aesthetics:SFE_LOGO_FLAME_.1 -> xensiv_pas:INFINEON_LOGO
- U$231, U$268: device output:#SDA#TX_#0 -> output:#GND_#0
- U$233: device output:#_SCL#0 -> output:#_RX#0
- U$236, U$274: device output:#_INT#0 -> output:#RX_#0
- U$239: device output:#I�C#0 -> output:#_SCL#0
- U$240, U$314, U$425: device SparkFun-Aesthetics:SFE_LOGO_FLAME_STOP_.1 -> output:#_GND#0
- U$241: device output:PWR0 -> output:#_3V3#0
- U$243, U$280: device output:#I#0 -> output:#_INT#0
- U$244: device output:#12VI_#0 -> output:#PSEL#0
- U$245: device output:#_12VIN#0 -> output:#I�C#0
- U$246, U$284: device output:#_EN#0 -> SparkFun-Aesthetics:SFE_LOGO_FLAME_STOP_.1
- U$248: device output:#_3V3#0 -> output:#U#0
- U$249: device output:#P_#0 -> output:#I#0
- U$250: device output:#_PWM#0 -> output:#12VI_#0
- U$251: device output:#PWM#0 -> output:#_12VIN#0
- U$253, U$290, U$291, U$328: device output:#_SDA#0 -> output:#_EN#0
- U$255: device output:#_SCL#0 -> output:#P_#0
- U$256: device output:PHOTOACOUSTIC0 -> output:#_PWM#0
- U$257: device output:SPECTROSCOPY0 -> output:#PWM#0
- U$258: device output:CO2_SENSOR0 -> output:#PWR#0
- U$260, U$297: device SparkFun-Aesthetics:SFE_LOGO_FLAME_.1 -> output:#_SDA#0
- U$261, U$299: device output:#GND_#0 -> output:#_SCL#0
- U$263: device output:#_TX#0 -> output:SPECTROSCOPY0
- U$264: device output:#_RX#0 -> output:CO2_SENSOR0
- U$265, U$303, U$417: device output:#_GND#0 -> output:PASCO2V010
- U$267: device output:#RX_#0 -> SparkFun-Aesthetics:SFE_LOGO_FLAME_.1
- U$270: device output:#_SCL#0 -> output:#_TX#0
- U$275: device output:#PSEL#0 -> output:#SDA#TX_#0
- U$277: device SparkFun-Aesthetics:SFE_LOGO_FLAME_STOP_.1 -> output:#_SCL#0
- U$278, U$352: device output:PWR0 -> output:#_GND#0
- U$279: device output:#U#0 -> output:#_3V3#0
- U$281, U$318: device output:#12VI_#0 -> output:#_INT#0
- U$282: device output:#_12VIN#0 -> output:#PSEL#0
- U$283, U$321: device output:#_EN#0 -> output:#I�C#0
- U$285: device output:#_3V3#0 -> output:PWR0
- U$286: device output:#P_#0 -> output:#U#0
- U$287: device output:#_PWM#0 -> output:#I#0
- U$288: device output:#PWM#0 -> output:#12VI_#0
- U$289: device output:#PWR#0 -> output:#_12VIN#0
- U$292: device output:#_SCL#0 -> output:#_3V3#0
- U$293: device output:PHOTOACOUSTIC0 -> output:#P_#0
- U$294: device output:SPECTROSCOPY0 -> output:#_PWM#0
- U$295: device output:CO2_SENSOR0 -> output:#PWM#0
- U$296: device output:PASCO2V010 -> output:#PWR#0
- U$298, U$335, U$336, U$373: device output:#GND_#0 -> output:#_SDA#0
- U$30, U$77: device output:#GND_#0 -> SparkFun-Aesthetics:SFE_LOGO_FLAME_.1
- U$300: device output:#_TX#0 -> output:PHOTOACOUSTIC0
- U$301: device output:#_RX#0 -> output:SPECTROSCOPY0
- U$302, U$340: device output:#_GND#0 -> output:CO2_SENSOR0
- U$304: device output:#RX_#0 -> xensiv_pas:INFINEON_LOGO
- U$305: device output:#SDA#TX_#0 -> SparkFun-Aesthetics:SFE_LOGO_FLAME_.1
- U$307, U$344: device output:#_SCL#0 -> output:#GND_#0
- U$309: device output:#_3V3#0 -> output:#_RX#0
- U$312: device output:#PSEL#0 -> output:#RX_#0
- U$313: device output:#I�C#0 -> output:#SDA#TX_#0
- U$315: device output:PWR0 -> output:#_SCL#0
- U$316, U$390: device output:#U#0 -> output:#_GND#0
- U$317: device output:#I#0 -> output:#_3V3#0
- U$319, U$356: device output:#_12VIN#0 -> output:#_INT#0
- U$320, U$358: device output:#_EN#0 -> output:#PSEL#0
- U$322: device output:#_3V3#0 -> SparkFun-Aesthetics:SFE_LOGO_FLAME_STOP_.1
- U$323: device output:#P_#0 -> output:PWR0
- U$324: device output:#_PWM#0 -> output:#U#0
- U$325: device output:#PWM#0 -> output:#I#0
- U$326: device output:#PWR#0 -> output:#12VI_#0
- U$327, U$365: device output:#_SDA#0 -> output:#_12VIN#0
- U$329, U$366: device output:#_SCL#0 -> output:#_EN#0
- U$330: device output:PHOTOACOUSTIC0 -> output:#_3V3#0
- U$331: device output:SPECTROSCOPY0 -> output:#P_#0
- U$332: device output:CO2_SENSOR0 -> output:#_PWM#0
- U$333: device output:PASCO2V010 -> output:#PWM#0
- U$334: device SparkFun-Aesthetics:SFE_LOGO_FLAME_.1 -> output:#PWR#0
- U$337: device output:#_TX#0 -> output:#_SCL#0
- U$338: device output:#_RX#0 -> output:PHOTOACOUSTIC0
- U$339, U$377: device output:#_GND#0 -> output:SPECTROSCOPY0
- U$341: device output:#RX_#0 -> output:PASCO2V010
- U$342: device output:#SDA#TX_#0 -> xensiv_pas:INFINEON_LOGO
- U$346: device output:#_3V3#0 -> output:#_TX#0
- U$347, U$385: device output:#_INT#0 -> output:#_RX#0
- U$350: device output:#I�C#0 -> output:#RX_#0
- U$351: device SparkFun-Aesthetics:SFE_LOGO_FLAME_STOP_.1 -> output:#SDA#TX_#0
- U$353: device output:#U#0 -> output:#_SCL#0
- U$354, U$428: device output:#I#0 -> output:#_GND#0
- U$355: device output:#12VI_#0 -> output:#_3V3#0
- U$357, U$394, U$395, U$432: device output:#_EN#0 -> output:#_INT#0
- U$359: device output:#_3V3#0 -> output:#I�C#0
- U$360: device output:#P_#0 -> SparkFun-Aesthetics:SFE_LOGO_FLAME_STOP_.1
- U$361: device output:#_PWM#0 -> output:PWR0
- U$362: device output:#PWM#0 -> output:#U#0
- U$363: device output:#PWR#0 -> output:#I#0
- U$364, U$402: device output:#_SDA#0 -> output:#12VI_#0
- U$367, U$404: device output:PHOTOACOUSTIC0 -> output:#_EN#0
- U$368: device output:SPECTROSCOPY0 -> output:#_3V3#0
- U$369: device output:CO2_SENSOR0 -> output:#P_#0
- U$370: device output:PASCO2V010 -> output:#_PWM#0
- U$371: device SparkFun-Aesthetics:SFE_LOGO_FLAME_.1 -> output:#PWM#0
- U$372, U$410: device output:#GND_#0 -> output:#PWR#0
- U$374, U$411: device output:#_TX#0 -> output:#_SDA#0
- U$375: device output:#_RX#0 -> output:#_SCL#0
- U$376, U$414: device output:#_GND#0 -> output:PHOTOACOUSTIC0
- U$378: device output:#RX_#0 -> output:CO2_SENSOR0
- U$379: device output:#SDA#TX_#0 -> output:PASCO2V010
- U$381: device output:#_SCL#0 -> SparkFun-Aesthetics:SFE_LOGO_FLAME_.1
- U$383, U$420: device output:#_3V3#0 -> output:#GND_#0
- U$384, U$422: device output:#_INT#0 -> output:#_TX#0
- U$388: device SparkFun-Aesthetics:SFE_LOGO_FLAME_STOP_.1 -> output:#RX_#0
- U$389: device output:PWR0 -> output:#SDA#TX_#0
- U$391: device output:#I#0 -> output:#_SCL#0
- U$392: device output:#12VI_#0 -> output:#_GND#0
- U$393: device output:#_12VIN#0 -> output:#_3V3#0
- U$396: device output:#_3V3#0 -> output:#PSEL#0
- U$397: device output:#P_#0 -> output:#I�C#0
- U$398: device output:#_PWM#0 -> SparkFun-Aesthetics:SFE_LOGO_FLAME_STOP_.1
- U$399: device output:#PWM#0 -> output:PWR0
- U$400: device output:#PWR#0 -> output:#U#0
- U$401, U$439: device output:#_SDA#0 -> output:#I#0
- U$403: device output:#_SCL#0 -> output:#_12VIN#0
- U$405, U$442: device output:SPECTROSCOPY0 -> output:#_EN#0
- U$406: device output:CO2_SENSOR0 -> output:#_3V3#0
- U$407: device output:PASCO2V010 -> output:#P_#0
- U$408: device SparkFun-Aesthetics:SFE_LOGO_FLAME_.1 -> output:#_PWM#0
- U$409: device output:#GND_#0 -> output:#PWM#0
- U$41, U$78: device output:#_TX#0 -> output:#GND_#0
- U$412: device output:#_RX#0 -> output:#_SDA#0
- U$413, U$49: device output:#_GND#0 -> output:#_SCL#0
- U$415: device output:#RX_#0 -> output:SPECTROSCOPY0
- U$416: device output:#SDA#TX_#0 -> output:CO2_SENSOR0
- U$418: device output:#_SCL#0 -> xensiv_pas:INFINEON_LOGO
- U$42: device output:#_RX#0 -> output:#_TX#0
- U$421: device output:#_INT#0 -> output:#GND_#0
- U$423: device output:#PSEL#0 -> output:#_RX#0
- U$426: device output:PWR0 -> output:#RX_#0
- U$427: device output:#U#0 -> output:#SDA#TX_#0
- U$429: device output:#12VI_#0 -> output:#_SCL#0
- U$430: device output:#_12VIN#0 -> output:#_GND#0
- U$431: device output:#_EN#0 -> output:#_3V3#0
- U$433: device output:#_3V3#0 -> output:#_INT#0
- U$434: device output:#P_#0 -> output:#PSEL#0
- U$435: device output:#_PWM#0 -> output:#I�C#0
- U$436: device output:#PWM#0 -> SparkFun-Aesthetics:SFE_LOGO_FLAME_STOP_.1
- U$437: device output:#PWR#0 -> output:PWR0
- U$438: device output:#_SDA#0 -> output:#U#0
- U$440: device output:#_SCL#0 -> output:#12VI_#0
- U$441: device output:PHOTOACOUSTIC0 -> output:#_12VIN#0
- U$443: device output:CO2_SENSOR0 -> output:#_EN#0
- U$444: device output:PASCO2V010 -> output:#_3V3#0
- U$45, U$82: device output:#RX_#0 -> output:#_GND#0
- U$46: device output:#SDA#TX_#0 -> output:#RX_#0
- U$51, U$89: device output:#_INT#0 -> output:#_3V3#0
- U$53, U$90: device output:#PSEL#0 -> output:#_INT#0
- U$54: device output:#I�C#0 -> output:#PSEL#0
- U$55: device SparkFun-Aesthetics:SFE_LOGO_FLAME_STOP_.1 -> output:#I�C#0
- U$56: device output:PWR0 -> SparkFun-Aesthetics:SFE_LOGO_FLAME_STOP_.1
- U$57: device output:#U#0 -> output:PWR0
- U$58: device output:#I#0 -> output:#U#0
- U$59: device output:#12VI_#0 -> output:#I#0
- U$60: device output:#_12VIN#0 -> output:#12VI_#0
- U$61, U$99: device output:#_EN#0 -> output:#_12VIN#0
- U$64: device output:#P_#0 -> output:#_3V3#0
- U$65: device output:#_PWM#0 -> output:#P_#0
- U$66: device output:#PWM#0 -> output:#_PWM#0
- U$67: device output:#PWR#0 -> output:#PWM#0
- U$71: device output:PHOTOACOUSTIC0 -> output:#_SCL#0
- U$72: device output:SPECTROSCOPY0 -> output:PHOTOACOUSTIC0
- U$73: device output:CO2_SENSOR0 -> output:SPECTROSCOPY0
- U$74: device output:PASCO2V010 -> output:CO2_SENSOR0
- U$75: device SparkFun-Aesthetics:SFE_LOGO_FLAME_.1 -> output:PASCO2V010
- U$85: device output:#_SCL#0 -> output:#SDA#TX_#0
- U$87: device output:#_3V3#0 -> output:#_SCL#0
- U$92: device SparkFun-Aesthetics:SFE_LOGO_FLAME_STOP_.1 -> output:#PSEL#0
- U$93: device output:PWR0 -> output:#I�C#0
- U$94: device output:#U#0 -> SparkFun-Aesthetics:SFE_LOGO_FLAME_STOP_.1
- U$95: device output:#I#0 -> output:PWR0
- U$96: device output:#12VI_#0 -> output:#U#0
- U$97: device output:#_12VIN#0 -> output:#I#0
- U10, U12, U14, U16, U18, U2, U20, U22, U24, U4, U6, U8: value LMR62421 -> AP3012
- moved U$227 154.2 mm to (142.2, 10.3), flipped to the bottom
- moved U$225 152.0 mm to (142.2, 13.5)
- moved U$226 151.6 mm to (142.2, 11.9), flipped to the bottom
- moved U$228 139.8 mm to (137.1, 37.4), flipped to the bottom
- moved U$223 139.2 mm to (143.5, 1.27), flipped to the bottom, turned to 90 degrees
- moved U$224 130.4 mm to (142.2, 15.0), flipped to the bottom
- moved U$418 48.4 mm to (111.2, 78.5), flipped to the bottom, turned to 0 degrees
- moved U$298 47.7 mm to (37.3, 42.4), flipped to the bottom, turned to 90 degrees
- moved U$335 47.7 mm to (63.2, 42.4), turned to 90 degrees
- moved U$261 45.6 mm to (14.0, 42.4), flipped to the bottom, turned to 90 degrees
- moved U$380 43.7 mm to (85.3, 78.5), flipped to the bottom, turned to 0 degrees
- moved U$266 43.2 mm to (7.58, 78.5)
- moved U$76 43.2 mm to (33.5, 37.4), flipped to the bottom
- moved U$23 43.0 mm to (7.58, 37.4), flipped to the bottom
- moved U$303 41.9 mm to (38.6, 51.4)
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